File: Power.kicad_sch (KiCad schematic)
At the start: 4 parts, among them U5 RT9013-33GB

Commit message: 优化接口
Parts:
- removed U5: RT9013-33GB, symbol User_Driver:RT9013-33GB
- added U4: RT9013-33GB, Package_TO_SOT_SMD:SOT-23-5, symbol User_Driver:RT9013-33GB
- C1, C2: footprint (none) -> Capacitor_SMD:C_0603_1608Metric_Pad1.08x0.95mm_HandSolder
- R3: footprint (none) -> Resistor_SMD:R_0603_1608Metric_Pad0.98x0.95mm_HandSolder
Connections:
- net +5V: now also U4.1 (VIN), U4.3 (EN)
- net 3V3: now also U4.5 (OUT)
- net GND: now also U4.2 (GND)
Other:
- moved on the sheet: C1, C2, R3
