File: ControlBoard.kicad_sch (KiCad schematic)
At the start: 9 parts, among them J1 Conn_02x06_Odd_Even, J2 Conn_02x06_Odd_Even, J3 Conn_02x03_Odd_Even, J5 Conn_01x06, J6 Conn_01x06, J7 Conn_01x02

Commit message: 优化接口
Parts:
- R5: value 0R -> NC; footprint (none) -> Resistor_SMD:R_0603_1608Metric_Pad0.98x0.95mm_HandSolder
- TP1, TP2: footprint (none) -> TestPoint:TestPoint_Pad_D1.0mm
Connections:
- net PWM1_CH3N is gone; now on net MOTOR1_U-: J1.12 (Pin_12)
- net PWM8_CH3N is gone; now on net MOTOR2_U-: J2.12 (Pin_12)
- net ADC1_BusCurr renamed busCurrent
- net ADC1_BusVol renamed BusVoltage
- net ADC1_U renamed MOTOR1_ADC_U
- net ADC1_V renamed MOTOR1_ADC_V
- net ADC1_W renamed MOTOR1_ADC_W
- net ADC2_U renamed MOTOR2_ADC_U
- net ADC2_V renamed MOTOR2_ADC_V
- net ADC2_W renamed MOTOR2_ADC_W
- net MCU_Part/PWM1_CH4 renamed MCU_Part/PA11_TIM1_CH4
- net MCU_Part/PWM8_CH4 renamed MCU_Part/PC9_TIM8_CH4
- net PWM1_CH1 renamed MOTOR1_U+
- net PWM1_CH1N renamed MOTOR1_U-
- net PWM1_CH2 renamed MOTOR1_V+
- net PWM1_CH2N renamed MOTOR1_V-
- net PWM1_CH3 renamed MOTOR1_W+
- net PWM8_CH1 renamed MOTOR2_U+
- net PWM8_CH1N renamed MOTOR2_U-
- net PWM8_CH2 renamed MOTOR2_V+
- net PWM8_CH2N renamed MOTOR2_V-
- net PWM8_CH3 renamed MOTOR2_W+
Other:
- sheet MCU_Part ports: added PA10_TIM1_CH3, PA11_TIM1_CH4, PA15_SPI3_CS, PA4_SPI1_CS, PA5_SPI1_SCK, PA6_SPI1_MISO, PA7_SPI1_MOSI, PA8_TIM1_CH1, PA9_TIM1_CH2, PB13_TIM1_CH1N, PB14_TIM1_CH2N, PB15_TIM1_CH3N, PB3_TIM8_CH1N, PB4_TIM8_CH2N, PB5_TIM8_CH3N, PC10_SPI3_SCK, PC11_SPI3_MISO, PC12_SPI3_MOSI, PC6_TIM8_CH1, PC7_TIM8_CH2, PC8_TIM8_CH3, PC9_TIM8_CH4; removed PWM1_CH1, PWM1_CH1N, PWM1_CH2, PWM1_CH2N, PWM1_CH3, PWM1_CH3N, PWM1_CH4, PWM8_CH1, PWM8_CH1N, PWM8_CH2, PWM8_CH2N, PWM8_CH3, PWM8_CH3N, PWM8_CH4, SPI1_CS, SPI1_MISO, SPI1_MOSI, SPI1_SCK, SPI3_CS, SPI3_MISO, SPI3_MOSI, SPI3_SCK
- moved on the sheet: J1, J2, J3, J5, J6, J7, R5, TP1, TP2

Commit message: 增加网表及PCB文件
Parts:
- removed J1, J2: Conn_02x06_Odd_Even, symbol Connector_Generic:Conn_02x06_Odd_Even
- added J1, J2: Conn_02x07_Odd_Even, Connector_PinSocket_1.27mm:PinSocket_2x07_P1.27mm_Vertical_SMD, symbol Connector_Generic:Conn_02x07_Odd_Even
- J3: footprint (none) -> Connector_IDC:IDC-Header_2x03_P2.54mm_Vertical_SMD
- J5, J6: footprint (none) -> Connector_JST:JST_SH_BM06B-SRSS-TB_1x06-1MP_P1.00mm_Vertical
- J7: footprint (none) -> Connector_JST:JST_SH_BM02B-SRSS-TB_1x02-1MP_P1.00mm_Vertical
Connections:
- net +5V: now also J2.9 (Pin_9)
- net 3.3V: now also J2.11 (Pin_11)
- net BusVoltage: now also J1.7 (Pin_7)
- net GND: now also J1.14 (Pin_14), J2.13 (Pin_13)
- net MOTOR1_ADC_U: now also J1.1 (Pin_1)
- net MOTOR1_ADC_V: now also J1.3 (Pin_3)
- net MOTOR1_ADC_W: now also J1.5 (Pin_5)
- net MOTOR1_U+: now also J1.2 (Pin_2)
- net MOTOR1_U-: now also J1.12 (Pin_12), J1.4 (Pin_4)
- net MOTOR1_V+: now also J1.6 (Pin_6)
- net MOTOR1_V-: now also J1.8 (Pin_8)
- net MOTOR1_W+: now also J1.10 (Pin_10)
- net MOTOR2_ADC_U: now also J2.1 (Pin_1)
- net MOTOR2_ADC_V: now also J2.3 (Pin_3)
- net MOTOR2_ADC_W: now also J2.5 (Pin_5)
- net MOTOR2_U+: now also J2.2 (Pin_2)
- net MOTOR2_U-: now also J2.12 (Pin_12), J2.4 (Pin_4)
- net MOTOR2_V+: now also J2.6 (Pin_6)
- net MOTOR2_V-: now also J2.8 (Pin_8)
- net MOTOR2_W+: now also J2.10 (Pin_10)
- net busCurrent: now also J1.9 (Pin_9)
- new net MOTOR1_BREAK: J1.11 (Pin_11)
- new net MOTOR2_BREAK: J2.7 (Pin_7)
